File: eda/psycho_badge/psycho_badge.kicad_pcb (KiCad board)
At the start: 2 copper layers, 152.4 x 101.6 mm, 74 parts, among them J1 Battery_Conn, J21 01x02, J22 01x02, SW1 SW_SPDT_SS12D00G, U1 ESP32-WEMOS-LOLIN32-LITE

Commit message: pcb updates
Routing:
- net GND: vias 0 -> 3
