File: eda/psycho_badge/psycho_badge_back.kicad_pcb (KiCad board)
At the start: 2 copper layers, 152.4 x 101.6 mm, 5 parts

Commit message: main badge pcb updates
Parts:
- added G***: LOGO, 0_badge:psycho_badge_rear_art, F.Cu at (140.6, 87.6)
- added G***: LOGO, 0_badge:scream_face_cu_back_55mx80mm, F.Cu at (141.0, 84.8)
- added G***: LOGO, 0_alt_bier:logo-alt_bier-900dpi-10x25mm-copper-front, F.Cu at (207.0, 116.5)
Other:
- board text added: "Batt Charging LED"
- board text added: "https://psycho.altbier.us"

Commit message: pcb updates
Parts:
- moved G*** 1.05 mm to (140.1, 84.3)
Changed lines of the file:
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@@
 	(footprint "0_badge:scream_face_cu_back_55mx80mm"
 		(layer "F.Cu")
-		(at 141 84.75)
+		(at 140.05 84.3)
 		(property "Reference" "G***"
 			(at 0.325 -38.425 0)
@@
 		)
 		(fill yes)
-		(layer "F.SilkS")
+		(layer "F.Mask")
 	)
 	(gr_circle
@@
 		)
 		(fill yes)
-		(layer "F.SilkS")
+		(layer "F.Mask")
 	)
 	(gr_circle
@@
 		)
 		(fill yes)
-		(layer "B.SilkS")
+		(layer "B.Mask")
 	)
 	(gr_circle
@@
 		)
 		(fill yes)
-		(layer "B.SilkS")
+		(layer "B.Mask")
 	)
 	(gr_line

Commit message: pcb updates... final?
Parts:
- added G***: LOGO, 0_org_logos:3000_Society_Logo_Front_20mmx11mm, F.Cu at (189.9, 123.7)
- added Lanyard: Lanyard_Hole, 0_local:Lanyard_Hole, F.Cu at (184.9, 41.4)
- added Lanyard: Lanyard_Hole, 0_local:Lanyard_Hole, F.Cu at (96.1, 41.4)
