File: eda/psycho_sao/psycho_sao_2.kicad_pcb (KiCad board)
At the start: 2 copper layers, 80.2 x 117.1 mm, 47 parts

Commit message: SB SAO final and code updates
Parts:
- added G***: LOGO, 0_badge:SB_silhouette_F_Silk_17mm, F.Cu at (129.8, 111.0)
- added G***: LOGO, 0_badge:SB_silhouette_F_Silk_17mm, F.Cu at (88.7, 111.0)
- added G***: LOGO, 0_badge:SB_silhouette_F_Silk_17mm, F.Cu at (111.3, 82.5)
- added G***: LOGO, 0_badge:SB_silhouette_F_Silk_17mm, F.Cu at (152.4, 82.5)
- G*** (x4): footprint 0_alt_bier:logo-alt_bier-1100dpi-8x21mm-back -> 0_alt_bier:logo-alt_bier-1200dpi-8x19mm-back
- moved D21 29.8 mm to (130.2, 50.3)
- moved D41 29.8 mm to (152.0, 143.2)
- moved D11 29.8 mm to (89.1, 50.3)
- moved D31 29.8 mm to (110.9, 143.2)
- moved Fold 29.7 mm to (130.2, 53.7)
- moved Fold 29.7 mm to (89.1, 53.7)
- moved REF** 29.7 mm to (89.1, 52.3)
- moved REF** 29.7 mm to (130.2, 52.3)
- moved REF** 29.6 mm to (152.0, 141.1)
- moved REF** 29.6 mm to (110.9, 141.1)
- moved Fold 29.4 mm to (110.9, 139.4)
- moved Fold 29.4 mm to (152.0, 139.4)
- moved D32 5.05 mm to (83.9, 126.2), turned to -90 degrees
- moved D42 5.05 mm to (125.0, 126.2), turned to -90 degrees
- moved D22 4.98 mm to (157.2, 67.3), turned to 90 degrees
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Routing:
- net Net-(D31-K): track 7.12 -> 38.5 mm
- net Net-(D41-K): track 7.12 -> 38.5 mm
- net Net-(D21-K): track 7.13 -> 38.5 mm
- net Net-(D11-K): track 7.13 -> 38.5 mm
- net +3.3V2: track 50.1 -> 70.2 mm
- net +3.3V3: track 50.1 -> 70.2 mm
- net +3.3V1: track 50.1 -> 70.2 mm
- net +3.3V: track 50.1 -> 70.2 mm
- net Net-(D32-K): track 24.3 -> 19.5 mm
- net Net-(D42-K): track 24.3 -> 19.5 mm
- net Net-(D22-K): track 24.2 -> 19.5 mm
- net Net-(D12-K): track 24.2 -> 19.5 mm
Other:
- board text added: "www.twitch.tv/skittishandbus"
